File: roshambo-pcb-smt.kicad_sch (KiCad schematic)
At the start: 49 parts, among them J1 Conn_01x06_Socket, J2 Conn_01x03_Pin, J3 Conn_01x03_Pin, Q1 2N7002, Q2 2N7002, Q3 2N7002, Q4 2N7002, Q5 2N7002, Q6 2N7002, Q7 2N7002, Q8 2N7002, Q9 2N7002, U1 Pico

Commit message: Updates
Parts:
- D1, D2, D3, D4, D5, D6, D7, D8, D9: footprint (none) -> LED_SMD:LED_0805_2012Metric
- J1: footprint (none) -> Connector_PinHeader_2.54mm:PinHeader_1x06_P2.54mm_Vertical
- J2, J3: footprint (none) -> Connector_PinHeader_2.54mm:PinHeader_1x03_P2.54mm_Vertical
- R1, R10, R11, R12, R13, R14, R15, R16, R17, R18, R19, R2, R20, R21, R22, R23, R24, R25, R26, R27, R3, R4, R5, R6, R7, R8, R9: footprint (none) -> Resistor_SMD:R_0603_1608Metric
Changed lines of the file:
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@@
       (effects (font (size 1.27 1.27)) (justify left))
     )
-    (property "Footprint" "" (at 140.716 114.554 90)
+    (property "Footprint" "Resistor_SMD:R_0603_1608Metric" (at 140.716 114.554 90)
       (effects (font (size 1.27 1.27)) hide)
     )
@@
       (effects (font (size 1.27 1.27)) (justify right))
     )
-    (property "Footprint" "" (at 153.67 90.17 0)
+    (property "Footprint" "LED_SMD:LED_0805_2012Metric" (at 153.67 90.17 0)
       (effects (font (size 1.27 1.27)) hide)
     )
@@
       (effects (font (size 1.27 1.27)) (justify left))
     )
-    (property "Footprint" "" (at 50.546 155.194 90)
+    (property "Footprint" "Resistor_SMD:R_0603_1608Metric" (at 50.546 155.194 90)
       (effects (font (size 1.27 1.27)) hide)
     )
@@
       (effects (font (size 1.27 1.27)) (justify right))
     )
-    (property "Footprint" "" (at 49.53 90.17 0)
+    (property "Footprint" "LED_SMD:LED_0805_2012Metric" (at 49.53 90.17 0)
       (effects (font (size 1.27 1.27)) hide)
     )
@@
       (effects (font (size 1.27 1.27)) (justify right))
     )
-    (property "Footprint" "" (at 106.68 90.17 0)
+    (property "Footprint" "LED_SMD:LED_0805_2012Metric" (at 106.68 90.17 0)
       (effects (font (size 1.27 1.27)) hide)
     )
@@
       (effects (font (size 1.27 1.27)) (justify right))
     )
-    (property "Footprint" "" (at 49.53 146.05 0)
+    (property "Footprint" "LED_SMD:LED_0805_2012Metric" (at 49.53 146.05 0)
       (effects (font (size 1.27 1.27)) hide)
     )
@@
       (effects (font (size 1.27 1.27)) (justify left))
     )
-    (property "Footprint" "" (at 36.576 57.404 90)
+    (property "Footprint" "Resistor_SMD:R_0603_1608Metric" (at 36.576 57.404 90)
       (effects (font (size 1.27 1.27)) hide)
     )
@@
       (effects (font (size 1.27 1.27)))
     )
-    (property "Footprint" "" (at 227.33 121.92 0)
+    (property "Footprint" "Connector_PinHeader_2.54mm:PinHeader_1x03_P2.54mm_Vertical" (at 227.33 121.92 0)
       (effects (font (size 1.27 1.27)) hide)
     )
@@
       (effects (font (size 1.27 1.27)) (justify left))
     )
-    (property "Footprint" "" (at 141.986 57.404 90)
+    (property "Footprint" "Resistor_SMD:R_0603_1608Metric" (at 141.986 57.404 90)
       (effects (font (size 1.27 1.27)) hide)
     )
@@
       (effects (font (size 1.27 1.27)))
     )
-    (property "Footprint" "" (at 87.884 109.474 90)
+    (property "Footprint" "Resistor_SMD:R_0603_1608Metric" (at 87.884 109.474 90)
       (effects (font (size 1.27 1.27)) hide)
     )
@@
       (effects (font (size 1.27 1.27)) (justify left))
     )
-    (property "Footprint" "" (at 107.696 155.194 90)
+    (property "Footprint" "Resistor_SMD:R_0603_1608Metric" (at 107.696 155.194 90)
       (effects (font (size 1.27 1.27)) hide)
     )
@@
       (effects (font (size 1.27 1.27)) (justify left))
     )
-    (property "Footprint" "" (at 155.956 42.164 90)
+    (property "Footprint" "Resistor_SMD:R_0603_1608Metric" (at 155.956 42.164 90)
       (effects (font (size 1.27 1.27)) hide)
     )
@@
       (effects (font (size 1.27 1.27)) (justify left))
     )
-    (property "Footprint" "" (at 93.726 57.404 90)
+    (property "Footprint" "Resistor_SMD:R_0603_1608Metric" (at 93.726 57.404 90)
       (effects (font (size 1.27 1.27)) hide)
     )
@@
       (effects (font (size 1.27 1.27)) (justify left))
     )
-    (property "Footprint" "" (at 154.686 155.194 90)
+    (property "Footprint" "Resistor_SMD:R_0603_1608Metric" (at 154.686 155.194 90)
       (effects (font (size 1.27 1.27)) hide)
     )
@@
       (effects (font (size 1.27 1.27)))
     )
-    (property "Footprint" "" (at 30.734 52.324 90)
+    (property "Footprint" "Resistor_SMD:R_0603_1608Metric" (at 30.734 52.324 90)
       (effects (font (size 1.27 1.27)) hide)
     )
@@
       (effects (font (size 1.27 1.27)))
     )
-    (property "Footprint" "" (at 30.734 165.354 90)
+    (property "Footprint" "Resistor_SMD:R_0603_1608Metric" (at 30.734 165.354 90)
       (effects (font (size 1.27 1.27)) hide)
     )
@@
       (effects (font (size 1.27 1.27)) (justify left))
     )
-    (property "Footprint" "" (at 107.696 42.164 90)
+    (property "Footprint" "Resistor_SMD:R_0603_1608Metric" (at 107.696 42.164 90)
       (effects (font (size 1.27 1.27)) hide)
     )
@@
       (effects (font (size 1.27 1.27)))
     )
-    (property "Footprint" "" (at 134.874 109.474 90)
+    (property "Footprint" "Resistor_SMD:R_0603_1608Metric" (at 134.874 109.474 90)
       (effects (font (size 1.27 1.27)) hide)
     )
@@
       (effects (font (size 1.27 1.27)) (justify right))
     )
-    (property "Footprint" "" (at 153.67 146.05 0)
+    (property "Footprint" "LED_SMD:LED_0805_2012Metric" (at 153.67 146.05 0)
       (effects (font (size 1.27 1.27)) hide)
     )
@@
       (effects (font (size 1.27 1.27)))
     )
-    (property "Footprint" "" (at 255.27 121.92 0)
+    (property "Footprint" "Connector_PinHeader_2.54mm:PinHeader_1x03_P2.54mm_Vertical" (at 255.27 121.92 0)
       (effects (font (size 1.27 1.27)) hide)
     )
@@
       (effects (font (size 1.27 1.27)) (justify left))
     )
-    (property "Footprint" "" (at 141.986 170.434 90)
+    (property "Footprint" "Resistor_SMD:R_0603_1608Metric" (at 141.986 170.434 90)
       (effects (font (size 1.27 1.27)) hide)
     )
@@
       (effects (font (size 1.27 1.27)))
     )
-    (property "Footprint" "" (at 30.734 109.474 90)
+    (property "Footprint" "Resistor_SMD:R_0603_1608Metric" (at 30.734 109.474 90)
       (effects (font (size 1.27 1.27)) hide)
     )
@@
       (effects (font (size 1.27 1.27)) (justify left))
     )
-    (property "Footprint" "" (at 36.576 170.434 90)
+    (property "Footprint" "Resistor_SMD:R_0603_1608Metric" (at 36.576 170.434 90)
       (effects (font (size 1.27 1.27)) hide)
     )
@@
       (effects (font (size 1.27 1.27)))
     )
-    (property "Footprint" "" (at 132.334 52.324 90)
+    (property "Footprint" "Resistor_SMD:R_0603_1608Metric" (at 132.334 52.324 90)
       (effects (font (size 1.27 1.27)) hide)
     )
@@
       (effects (font (size 1.27 1.27)) (justify left))
     )
-    (property "Footprint" "" (at 50.546 99.314 90)
+    (property "Footprint" "Resistor_SMD:R_0603_1608Metric" (at 50.546 99.314 90)
       (effects (font (size 1.27 1.27)) hide)
     )
@@
       (effects (font (size 1.27 1.27)))
     )
-    (property "Footprint" "" (at 85.344 52.324 90)
+    (property "Footprint" "Resistor_SMD:R_0603_1608Metric" (at 85.344 52.324 90)
       (effects (font (size 1.27 1.27)) hide)
     )
@@
       (effects (font (size 1.27 1.27)) (justify left))
     )
-    (property "Footprint" "" (at 154.686 99.314 90)
+    (property "Footprint" "Resistor_SMD:R_0603_1608Metric" (at 154.686 99.314 90)
       (effects (font (size 1.27 1.27)) hide)
     )
@@
       (effects (font (size 1.27 1.27)) (justify left))
     )
-    (property "Footprint" "" (at 107.696 99.314 90)
+    (property "Footprint" "Resistor_SMD:R_0603_1608Metric" (at 107.696 99.314 90)
       (effects (font (size 1.27 1.27)) hide)
     )
@@
       (effects (font (size 1.27 1.27)) (justify left))
     )
-    (property "Footprint" "" (at 93.726 114.554 90)
+    (property "Footprint" "Resistor_SMD:R_0603_1608Metric" (at 93.726 114.554 90)
       (effects (font (size 1.27 1.27)) hide)
     )
@@
       (effects (font (size 1.27 1.27)) (justify right))
     )
-    (property "Footprint" "" (at 49.53 33.02 0)
+    (property "Footprint" "LED_SMD:LED_0805_2012Metric" (at 49.53 33.02 0)
       (effects (font (size 1.27 1.27)) hide)
     )
@@
       (effects (font (size 1.27 1.27)) (justify left))
     )
-    (property "Footprint" "" (at 50.546 42.164 90)
+    (property "Footprint" "Resistor_SMD:R_0603_1608Metric" (at 50.546 42.164 90)
       (effects (font (size 1.27 1.27)) hide)
     )
@@
       (effects (font (size 1.27 1.27)) (justify left))
     )
-    (property "Footprint" "" (at 36.576 114.554 90)
+    (property "Footprint" "Resistor_SMD:R_0603_1608Metric" (at 36.576 114.554 90)
       (effects (font (size 1.27 1.27)) hide)
     )
@@
       (effects (font (size 1.27 1.27)) (justify left))
     )
-    (property "Footprint" "" (at 93.726 170.434 90)
+    (property "Footprint" "Resistor_SMD:R_0603_1608Metric" (at 93.726 170.434 90)
       (effects (font (size 1.27 1.27)) hide)
     )
@@
       (effects (font (size 1.27 1.27)))
     )
-    (property "Footprint" "" (at 136.144 165.354 90)
+    (property "Footprint" "Resistor_SMD:R_0603_1608Metric" (at 136.144 165.354 90)
       (effects (font (size 1.27 1.27)) hide)
     )
@@
       (effects (font (size 1.27 1.27)) (justify right))
     )
-    (property "Footprint" "" (at 106.68 146.05 0)
+    (property "Footprint" "LED_SMD:LED_0805_2012Metric" (at 106.68 146.05 0)
       (effects (font (size 1.27 1.27)) hide)
     )
@@
       (effects (font (size 1.27 1.27)) (justify right))
     )
-    (property "Footprint" "" (at 154.94 33.02 0)
+    (property "Footprint" "LED_SMD:LED_0805_2012Metric" (at 154.94 33.02 0)
       (effects (font (size 1.27 1.27)) hide)
     )
@@
       (effects (font (size 1.27 1.27)))
     )
-    (property "Footprint" "" (at 87.884 165.354 90)
+    (property "Footprint" "Resistor_SMD:R_0603_1608Metric" (at 87.884 165.354 90)
       (effects (font (size 1.27 1.27)) hide)
     )
@@
       (effects (font (size 1.27 1.27)) (justify right))
     )
-    (property "Footprint" "" (at 106.68 33.02 0)
+    (property "Footprint" "LED_SMD:LED_0805_2012Metric" (at 106.68 33.02 0)
       (effects (font (size 1.27 1.27)) hide)
     )
@@
       (effects (font (size 1.27 1.27)) (justify left))
     )
-    (property "Footprint" "" (at 196.85 121.92 0)
-      (effects (font (size 1.27 1.27)) hide)
-    )
+    (property "Footprint" "Connector_PinHeader_2.54mm:PinHeader_1x06_P2.54mm_Vertical" (at 196.85 121.92 0)
+      (effects (font (size 1.27 1.27)) hide)
+    )

Commit message: More progress on the layout
Parts:
- D1, D2, D3, D4, D5, D6, D7, D8, D9: footprint LED_SMD:LED_0805_2012Metric -> LED_SMD:LED_0603_1608Metric
- R1, R10, R11, R12, R13, R14, R15, R16, R17, R18, R19, R2, R20, R21, R22, R23, R24, R25, R26, R27, R3, R4, R5, R6, R7, R8, R9: footprint Resistor_SMD:R_0603_1608Metric -> Resistor_SMD:R_0402_1005Metric
Connections:
- net GND: no longer Q9.1 (G), R24.2, R27.1
- new net: Q9.1 (G), R24.2, R27.1

Commit message: Released to Production
Parts:
- D1, D4, D7: value LED -> RED
- D2, D5, D9: value LED -> GREEN
- D3, D6: value LED -> BLUE
- D8: value LED -> YELLOW
- R1, R10, R19, R20: value 47 -> 150
- R11, R2, R21: value 47 -> 40
- R12, R3: value 47 -> 88
Changed lines of the file:
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@@
       (effects (font (size 1.27 1.27)) (justify right))
     )
-    (property "Value" "LED" (at 156.21 90.17 90)
+    (property "Value" "BLUE" (at 156.21 90.17 90)
       (effects (font (size 1.27 1.27)) (justify right))
     )
@@
       (effects (font (size 1.27 1.27)) (justify left))
     )
-    (property "Value" "47" (at 52.07 156.21 0)
+    (property "Value" "150" (at 52.07 156.21 0)
       (effects (font (size 1.27 1.27)) (justify left))
     )
@@
       (effects (font (size 1.27 1.27)) (justify right))
     )
-    (property "Value" "LED" (at 53.34 93.0275 90)
+    (property "Value" "RED" (at 53.34 93.0275 90)
       (effects (font (size 1.27 1.27)) (justify right))
     )
@@
       (effects (font (size 1.27 1.27)) (justify right))
     )
-    (property "Value" "LED" (at 110.49 93.0275 90)
+    (property "Value" "GREEN" (at 110.49 93.0275 90)
       (effects (font (size 1.27 1.27)) (justify right))
     )
@@
     )
   )
-  (symbol (lib_id "power:+5V") (at 49.53 25.4 0) (unit 1)
-    (in_bom yes) (on_board yes) (dnp no) (fields_autoplaced)
-    (property "Reference" "#PWR02" (at 49.53 29.21 0)
-      (effects (font (size 1.27 1.27)) hide)
-    )
-    (property "Value" "+5V" (at 49.53 20.32 0)
-      (effects (font (size 1.27 1.27)))
-    )
-    (property "Footprint" "" (at 49.53 25.4 0)
-      (effects (font (size 1.27 1.27)) hide)
-    )
-    (property "Datasheet" "" (at 49.53 25.4 0)
-      (effects (font (size 1.27 1.27)) hide)
-    )
-    (pin "1")
-    (instances
-      (project "roshambo-pcb-smt"
-        (path "/603bd549-5ff3-45c4-94a9-865018e03ed8"
-          (reference "#PWR02") (unit 1)
-        )
-      )
-    )
-  )
   (symbol (lib_id "Device:LED") (at 49.53 146.05 90) (unit 1)
     (in_bom yes) (on_board yes) (dnp no) (fields_autoplaced)
@@
       (effects (font (size 1.27 1.27)) (justify right))
     )
-    (property "Value" "LED" (at 53.34 148.9075 90)
+    (property "Value" "RED" (at 53.34 148.9075 90)
       (effects (font (size 1.27 1.27)) (justify right))
     )
@@
       (effects (font (size 1.27 1.27)) (justify left))
     )
-    (property "Value" "47" (at 109.22 156.21 0)
+    (property "Value" "150" (at 109.22 156.21 0)
       (effects (font (size 1.27 1.27)) (justify left))
     )
@@
       (effects (font (size 1.27 1.27)) (justify left))
     )
-    (property "Value" "47" (at 157.48 43.18 0)
+    (property "Value" "88" (at 157.48 43.18 0)
       (effects (font (size 1.27 1.27)) (justify left))
     )
@@
       (effects (font (size 1.27 1.27)) (justify left))
     )
-    (property "Value" "47" (at 156.21 156.21 0)
+    (property "Value" "40" (at 156.21 156.21 0)
       (effects (font (size 1.27 1.27)) (justify left))
     )
@@
       (effects (font (size 1.27 1.27)) (justify left))
     )
-    (property "Value" "47" (at 109.22 43.18 0)
+    (property "Value" "40" (at 109.22 43.18 0)
       (effects (font (size 1.27 1.27)) (justify left))
     )
@@
       (effects (font (size 1.27 1.27)) (justify right))
     )
-    (property "Value" "LED" (at 157.48 148.9075 90)
+    (property "Value" "GREEN" (at 157.48 148.9075 90)
       (effects (font (size 1.27 1.27)) (justify right))
     )
@@
         (path "/603bd549-5ff3-45c4-94a9-865018e03ed8"
           (reference "#PWR011") (unit 1)
+        )
+      )
+    )
+  )
+  (symbol (lib_id "power:+5V") (at 49.53 25.4 0) (unit 1)
+    (in_bom yes) (on_board yes) (dnp no) (fields_autoplaced)
+    (property "Reference" "#PWR02" (at 49.53 29.21 0)
+      (effects (font (size 1.27 1.27)) hide)
+    )
+    (property "Value" "+5V" (at 49.53 20.32 0)
+      (effects (font (size 1.27 1.27)))
+    )
+    (property "Footprint" "" (at 49.53 25.4 0)
+      (effects (font (size 1.27 1.27)) hide)
+    )
+    (property "Datasheet" "" (at 49.53 25.4 0)
+      (effects (font (size 1.27 1.27)) hide)
+    )
+    (pin "1")
+    (instances
+      (project "roshambo-pcb-smt"
+        (path "/603bd549-5ff3-45c4-94a9-865018e03ed8"
+          (reference "#PWR02") (unit 1)
         )
       )
@@
       (effects (font (size 1.27 1.27)) (justify left))
     )
-    (property "Value" "47" (at 52.07 100.33 0)
+    (property "Value" "150" (at 52.07 100.33 0)
       (effects (font (size 1.27 1.27)) (justify left))
     )
@@
       (effects (font (size 1.27 1.27)) (justify left))
     )
-    (property "Value" "47" (at 156.21 100.33 0)
+    (property "Value" "88" (at 156.21 100.33 0)
       (effects (font (size 1.27 1.27)) (justify left))
     )
@@
       (effects (font (size 1.27 1.27)) (justify left))
     )
-    (property "Value" "47" (at 109.22 100.33 0)
+    (property "Value" "40" (at 109.22 100.33 0)
       (effects (font (size 1.27 1.27)) (justify left))
     )
@@
       (effects (font (size 1.27 1.27)) (justify right))
     )
-    (property "Value" "LED" (at 53.34 35.8775 90)
+    (property "Value" "RED" (at 53.34 35.8775 90)
       (effects (font (size 1.27 1.27)) (justify right))
     )
@@
       (effects (font (size 1.27 1.27)) (justify left))
     )
-    (property "Value" "47" (at 52.07 43.18 0)
+    (property "Value" "150" (at 52.07 43.18 0)
       (effects (font (size 1.27 1.27)) (justify left))
     )
@@
       (effects (font (size 1.27 1.27)) (justify right))
     )
-    (property "Value" "LED" (at 110.49 148.9075 90)
+    (property "Value" "YELLOW" (at 110.49 148.9075 90)
       (effects (font (size 1.27 1.27)) (justify right))
     )
@@
       (effects (font (size 1.27 1.27)) (justify right))
     )
-    (property "Value" "LED" (at 158.75 35.8775 90)
+    (property "Value" "BLUE" (at 158.75 35.8775 90)
       (effects (font (size 1.27 1.27)) (justify right))
     )
@@
       (effects (font (size 1.27 1.27)) (justify right))
     )
-    (property "Value" "LED" (at 110.49 35.8775 90)
-      (effects (font (size 1.27 1.27)) (justify right))
-    )
+    (property "Value" "GREEN" (at 110.49 35.8775 90)
+      (effects (font (size 1.27 1.27)) (justify right))
+    )
